File: schematics/LIA-board/dac.kicad_sch (KiCad schematic)
At the start: 23 parts, among them IC2 INA190, IC3 INA190, IC4 INA190, IC5 INA190, U15 DAC80508, U16 OPA2196xD, U17 OPA2196xD

Commit message: commit before changing the oscillator implementation
Connections:
- net +5VA: now also U15.7 (VDD); no longer C37.2, U16.8 (V+)
- net GMOS_Imeas1: no longer IC3.6 (OUT)
- net VDDA: now reaches IC4.3 (VS)
- net VDDA: now also IC2.3 (VS), IC3.3 (VS), IC5.3 (VS)
- net +3V3_D: now reaches U15.16 (VIO)
- new net +5VP: C37.2, U16.8 (V+)
- new net GMOS_Imeas0: IC3.6 (OUT)

Commit message: commit before changing LIA
Parts:
- removed IC4, IC5: INA190, symbol CERN:INA190AxIDCK
- R25: renamed from R45; value 15 -> 330k
- R31: renamed from R46; value 15 -> 330k
- renumbered C37 to C23, C39 to C24, C38 to C25, C40 to C26, IC2 to IC1, R36 to R20, R41 to R21, R35 to R22, R39 to R23, R43 to R24, R37 to R26, R42 to R27, R38 to R28, R40 to R29, R44 to R30, U17 to U10, U15 to U8, U16 to U9
Connections:
- net DAC6: now also R23.2
- net DAC7: now also R29.2
- net GMOS_Vadj0: now also R26.1
- net GMOS_Vadj1: now also R20.1
- net GND: no longer R23.2, R29.2
- net at IC3.4 (IN+), R30.2, U9.7: no longer R26.1
- net at IC1.4 (IN+), R24.2, U9.1: no longer R20.1
- net dac_cs: now reaches U8.12 (~{CS})
- net spi_clk: now reaches U8.13 (SCLK)
- net spi_mosi: now reaches U8.14 (SDI)
- net spi_miso: now reaches U8.15 (SDO/~{ALARM})
- net DAC4 renamed GMOS_Vadj4
- net DAC5 renamed GMOS_Vadj5
Other:
- moved on the sheet: R21, R23, R25, R27, R29, R31, U10A, U10B
