File: schematics/LIA-board/excitation.kicad_sch (KiCad schematic)
At the start: 17 parts, among them U13 OPA2196xD

Commit message: commit before changing LIA
Parts:
- renumbered C28 to C1, C36 to C2, C27 to C3, C41 to C4, C29 to C5, C48 to C6, C42 to C7, C47 to C8, R57 to R1, R54 to R2, R55 to R3, R56 to R4, R61 to R5, R58 to R6, R59 to R7, R60 to R8, U13 to U1
Connections:
- net mcu_cos is gone; now on net mcu_sin: R6.1
- net Exct0: now reaches C1.2, R1.2, U1.1
- net at C6.1, R7.2: now also U1.6 (-); no longer U1.5 (+)
- net Exct1: now reaches C6.2, R5.2, U1.7
- net at C8.2, R8.2: now also U1.5 (+); no longer U1.6 (-)
- net gate_vadjust renamed ext0_vadj
- net ext0_vadj: no longer R8.1
- new net ext1_vadj: R8.1
Other:
- moved on the sheet: C1, C2, C3, C4, C5, C6, C7, C8, R1, R2, R3, R4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
