File: schematics/LIA-board/GMOS_MUX.kicad_sch (KiCad schematic)
At the start: 0 parts

Commit message: net naming pass, upper case sheet files
Parts:
- added J3: DIP40_J19, Package_DIP:DIP-40_W15.24mm, symbol device_libraries:DIP40_J19
- added R38: 100k, SparkFun-Resistor:R_0603_1608Metric, symbol SparkFun:R
- added R54, R55: 18k, SparkFun-Resistor:R_0603_1608Metric, symbol SparkFun:R
- added R56, R57: 1k, SparkFun-Resistor:R_0603_1608Metric, symbol SparkFun:R
- added U20, U21: TMUX1109PW, Package_SO:TSSOP-16_4.4x5mm_P0.65mm, symbol device_libraries:TMUX1109PW
Connections:
- new net: J3.14 (NC), J3.26 (NC), J3.27 (NC), J3.34 (NC), J3.35 (NC), J3.7 (NC)
- new net +5VA: J3.15 (VDD), J3.36 (VDD), U20.14 (VDD), U21.14 (VDD)
- new net GND: J3.1 (S3), J3.13 (S1), J3.16 (HN1), J3.2 (HN3), J3.20 (S6), J3.21 (HN6), J3.25 (S5), J3.28 (GND), J3.29 (HN5), J3.33 (S4), J3.37 (HN4), J3.6 (S2), J3.8 (GND), J3.9 (HN2), R38.2, R54.2, R55.2, R56.2, R57.2, U20.15 (GND), U20.3 (VSS), U21.15 (GND), U21.3 (VSS)
- new net active_cal: R54.1, U20.7 (S4A)
- new net active_drain_force: U21.8 (DA)
- new net active_gate_voltage: J3.19 (G6), J3.24 (G5), J3.32 (G4)
- new net active_heater_cal: R56.1, R57.1, U20.10 (S4B), U21.10 (S4B)
- new net active_heater_force: U21.9 (DB)
- new net blind_cal: R55.1, U21.7 (S4A)
- new net blind_drain_force: U20.8 (DA)
- new net blind_gate_voltage: J3.12 (G1), J3.40 (G3), J3.5 (G2)
- new net blind_heater_force: U20.9 (DB)
- new net ch_sel_0: U20.1 (A0)
- new net ch_sel_1: U20.16 (A1)
- new net ch_sel_2: U21.1 (A0)
- new net ch_sel_3: U21.16 (A1)
- new net drain_1: J3.17 (D1), U20.4 (S1A)
- new net drain_2: J3.10 (D2), U20.5 (S2A)
- new net drain_3: J3.3 (D3), U20.6 (S3A)
- new net drain_4: J3.38 (D4), U21.4 (S1A)
- new net drain_5: J3.30 (D5), U21.5 (S2A)
- new net drain_6: J3.22 (D6), U21.6 (S3A)
- new net heater_1: J3.11 (HP1), U20.13 (S1B)
- new net heater_2: J3.4 (HP2), U20.12 (S2B)
- new net heater_3: J3.39 (HP3), U20.11 (S3B)
- new net heater_4: J3.31 (HP4), U21.13 (S1B)
- new net heater_5: J3.23 (HP5), U21.12 (S2B)
- new net heater_6: J3.18 (HP6), U21.11 (S3B)
- new net mux_en: R38.1, U20.2 (EN), U21.2 (EN)
