File: schematics/LIA-board/GMOS_MUX.kicad_sch (KiCad schematic)
At the start: 8 parts, among them J3 DIP40_J19, U20 TMUX1109PW, U21 TMUX1109PW

Commit message: changes to scematic
Connections:
- net active_drain_force renamed DRN_B
- net active_gate_voltage renamed GATE_B
- net active_heater_force renamed HTR_B
- net blind_drain_force renamed DRN_A
- net blind_gate_voltage renamed GATE_A
- net blind_heater_force renamed HTR_A
- net ch_sel_0 renamed MUXA_A0
- net ch_sel_1 renamed MUXA_A1
- net ch_sel_2 renamed MUXB_A0
- net ch_sel_3 renamed MUXB_A1
- net mux_en renamed MUX_EN
Changed lines of the file:
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@@
 		)
 	)
-	(label "ch_sel_1"
+	(label "MUXA_A1"
 		(at 81.28 55.88 0)
 		(effects
@@
 		)
 	)
-	(label "ch_sel_3"
+	(label "MUXB_A1"
 		(at 81.28 134.62 0)
 		(effects
@@
 		)
 	)
-	(label "ch_sel_0"
+	(label "MUXA_A0"
 		(at 81.28 52.07 0)
 		(effects
@@
 		)
 	)
-	(label "ch_sel_2"
+	(label "MUXB_A0"
 		(at 81.28 130.81 0)
 		(effects
@@
 		)
 	)
-	(hierarchical_label "active_gate_voltage"
+	(hierarchical_label "GATE_B"
 		(shape input)
 		(at 161.29 52.07 180)
@@
 		)
 	)
-	(hierarchical_label "active_drain_force"
+	(hierarchical_label "DRN_B"
 		(shape input)
 		(at 39.37 151.13 180)
@@
 		)
 	)
-	(hierarchical_label "mux_en"
+	(hierarchical_label "MUX_EN"
 		(shape input)
 		(at 38.1 20.32 180)
@@
 		)
 	)
-	(hierarchical_label "active_heater_force"
+	(hierarchical_label "HTR_B"
 		(shape input)
 		(at 39.37 168.91 180)
@@
 		)
 	)
-	(hierarchical_label "blind_gate_voltage"
+	(hierarchical_label "GATE_A"
 		(shape input)
 		(at 161.29 58.42 180)
@@
 		)
 	)
-	(hierarchical_label "blind_heater_force"
+	(hierarchical_label "HTR_A"
 		(shape input)
 		(at 39.37 90.17 180)
@@
 		)
 	)
-	(hierarchical_label "ch_sel_[0..3]"
+	(hierarchical_label "{MUXA_A0 MUXA_A1 MUXB_A0 MUXB_A1}"
 		(shape input)
 		(at 38.1 25.4 180)
@@
 		)
 	)
-	(hierarchical_label "blind_drain_force"
+	(hierarchical_label "DRN_A"
 		(shape input)
 		(at 39.37 72.39 180)
