File: schematics/LIA-board/ADC.kicad_sch (KiCad schematic)
At the start: 1 part, among them U7 ADS1220xPW

Commit message: changes to scematic
Connections:
- net adc_cs renamed ADC_CS
- net spi_clk renamed SPI_SCK
- net spi_miso renamed SPI_MISO
- net spi_mosi renamed SPI_MOSI
Changed lines of the file:
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@@
 		)
 	)
-	(hierarchical_label "spi_miso"
+	(hierarchical_label "SPI_MISO"
 		(shape output)
 		(at 184.15 81.28 0)
@@
 		)
 	)
-	(hierarchical_label "spi_mosi"
+	(hierarchical_label "SPI_MOSI"
 		(shape input)
 		(at 184.15 77.47 0)
@@
 		)
 	)
-	(hierarchical_label "spi_clk"
+	(hierarchical_label "SPI_SCK"
 		(shape input)
 		(at 184.15 73.66 0)
@@
 		)
 	)
-	(hierarchical_label "adc_cs"
+	(hierarchical_label "ADC_CS"
 		(shape input)
 		(at 184.15 85.09 0)
