File: schematics/LIA-board/ANALOG.kicad_sch (KiCad schematic)
At the start: 0 parts

Commit message: changes to scematic
Other:
- sheet Excitation: file excitation.kicad_sch -> EXCITATION.kicad_sch
- sheet Excitation ports: added EXC_DAC, GATE_DC_A, GATE_DC_B, {GATE_A GATE_B}; removed Exct[0..1], ext0_vadj, ext1_vadj, mcu_sin
- sheet GMOS_soc: file gmos_mux2.kicad_sch -> GMOS_MUX.kicad_sch
- sheet GMOS_soc ports: added DRN_A, DRN_B, GATE_A, GATE_B, HTR_A, HTR_B, MUX_EN, {MUXA_A0 MUXA_A1 MUXB_A0 MUXB_A1}; removed active_drain_force, active_gate_voltage, active_heater_force, blind_drain_force, blind_gate_voltage, blind_heater_force, ch_sel_[0..3], mux_en
- sheet LIA_FE: file lia_fe.kicad_sch -> LIA_FE.kicad_sch
- sheet LIA_FE ports: added DRN_A, DRN_B, REF_X, REF_Y, X_OUT, Y_OUT; removed X_chop, X_readout, Y_chop, Y_readout, active_readout, blind_readout
Changed lines of the file:
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@@
 		)
 	)
-	(label "Exct1"
+	(label "GATE_A"
 		(at 105.41 88.9 180)
 		(effects
@@
 		)
 	)
-	(label "Exct0"
+	(label "GATE_B"
 		(at 105.41 83.82 180)
 		(effects
@@
 		)
 	)
-	(hierarchical_label "ch_sel_[0..3]"
+	(hierarchical_label "{MUXA_A0 MUXA_A1 MUXB_A0 MUXB_A1}"
 		(shape input)
 		(at 57.15 54.61 180)
@@
 		)
 	)
-	(hierarchical_label "X_chop"
+	(hierarchical_label "REF_X"
 		(shape input)
 		(at 148.59 109.22 180)
@@
 		)
 	)
-	(hierarchical_label "Vheater_blind"
+	(hierarchical_label "HTR_A"
 		(shape input)
 		(at 57.15 48.26 180)
@@
 		)
 	)
-	(hierarchical_label "Vheater_active"
+	(hierarchical_label "HTR_B"
 		(shape input)
 		(at 57.15 43.18 180)
@@
 		)
 	)
-	(hierarchical_label "mux_en"
+	(hierarchical_label "MUX_EN"
 		(shape input)
 		(at 57.15 59.69 180)
@@
 		)
 	)
-	(hierarchical_label "Y_readout"
+	(hierarchical_label "Y_OUT"
 		(shape output)
 		(at 195.58 81.28 0)
@@
 		)
 	)
-	(hierarchical_label "Vdrain_active"
+	(hierarchical_label "DRN_B"
 		(shape input)
 		(at 57.15 33.02 180)
@@
 		)
 	)
-	(hierarchical_label "X_readout"
+	(hierarchical_label "X_OUT"
 		(shape output)
 		(at 195.58 68.58 0)
@@
 		)
 	)
-	(hierarchical_label "Vdrain_blind"
+	(hierarchical_label "DRN_A"
 		(shape input)
 		(at 57.15 38.1 180)
@@
 		)
 	)
-	(hierarchical_label "Y_chop"
+	(hierarchical_label "REF_Y"
 		(shape input)
 		(at 148.59 113.03 180)
@@
 		)
 	)
-	(hierarchical_label "ext1_vadj"
+	(hierarchical_label "GATE_DC_A"
 		(shape input)
 		(at 55.88 88.9 180)
@@
 		)
 	)
-	(hierarchical_label "mcu_sin_ref"
+	(hierarchical_label "EXC_DAC"
 		(shape input)
 		(at 55.88 68.58 180)
@@
 		)
 	)
-	(hierarchical_label "ext0_vadj"
+	(hierarchical_label "GATE_DC_B"
 		(shape input)
 		(at 55.88 83.82 180)
@@
 			)
 		)
-		(property "Sheetfile" "gmos_mux2.kicad_sch"
+		(property "Sheetfile" "GMOS_MUX.kicad_sch"
 			(at 107.95 94.5646 0)
 			(show_name no)
@@
 			)
 		)
-		(pin "active_drain_force" input
+		(pin "DRN_B" input
 			(at 107.95 33.02 180)
 			(effects
@@
 			)
 		)
-		(pin "blind_drain_force" input
+		(pin "DRN_A" input
 			(at 107.95 38.1 180)
 			(effects
@@
 			)
 		)
-		(pin "active_gate_voltage" input
+		(pin "GATE_B" input
 			(at 107.95 83.82 180)
 			(effects
@@
 			)
 		)
-		(pin "blind_gate_voltage" input
+		(pin "GATE_A" input
 			(at 107.95 88.9 180)
 			(effects
@@
 			)
 		)
-		(pin "active_heater_force" input
+		(pin "HTR_B" input
 			(at 107.95 43.18 180)
 			(effects
@@
 			)
 		)
-		(pin "blind_heater_force" input
+		(pin "HTR_A" input
 			(at 107.95 48.26 180)
 			(effects
@@
 			)
 		)
-		(pin "ch_sel_[0..3]" input
+		(pin "{MUXA_A0 MUXA_A1 MUXB_A0 MUXB_A1}" input
 			(at 107.95 54.61 180)
 			(effects
@@
 			)
 		)
-		(pin "mux_en" input
+		(pin "MUX_EN" input
 			(at 107.95 59.69 180)
 			(effects
@@
 			)
 		)
-		(property "Sheetfile" "lia_fe.kicad_sch"
+		(property "Sheetfile" "LIA_FE.kicad_sch"
 			(at 158.75 117.4246 0)
 			(show_name no)
@@
 			)
 		)
-		(pin "active_readout" input
+		(pin "DRN_B" input
 			(at 158.75 76.2 180)
 			(effects
@@
 			)
 		)
-		(pin "blind_readout" input
+		(pin "DRN_A" input
 			(at 158.75 72.39 180)
 			(effects
@@
 			)
 		)
-		(pin "X_readout" output
+		(pin "X_OUT" output
 			(at 187.96 68.58 0)
 			(effects
@@
 			)
 		)
-		(pin "Y_readout" output
+		(pin "Y_OUT" output
 			(at 187.96 81.28 0)
 			(effects
@@
 			)
 		)
-		(pin "X_chop" input
+		(pin "REF_X" input
 			(at 158.75 109.22 180)
 			(effects
@@
 			)
 		)
-		(pin "Y_chop" input
+		(pin "REF_Y" input
 			(at 158.75 113.03 180)
 			(effects
@@
 			)
 		)
-		(property "Sheetfile" "excitation.kicad_sch"
+		(property "Sheetfile" "EXCITATION.kicad_sch"
 			(at 66.04 94.5646 0)
 			(show_name no)
@@
 			)
 		)
-		(pin "mcu_sin" input
+		(pin "EXC_DAC" input
 			(at 66.04 68.58 180)
 			(effects
@@
 			)
 		)
-		(pin "Exct[0..1]" output
+		(pin "{GATE_A GATE_B}" output
 			(at 91.44 76.2 0)
 			(effects
@@
 			)
 		)
-		(pin "ext0_vadj" input
+		(pin "GATE_DC_B" input
 			(at 66.04 83.82 180)
 			(effects
@@
 			)
 		)
-		(pin "ext1_vadj" input
+		(pin "GATE_DC_A" input
 			(at 66.04 88.9 180)
 			(effects
