File: schematics/LIA-board/CONNECTORS.kicad_sch (KiCad schematic)
At the start: 6 parts, among them J1 USB_C_Receptacle_PowerOnly_6P, J4 ${FAMILY}, J5 Conn_01x05_Pin, J6 Conn_01x05_Pin

Commit message: changes to scematic
Connections:
- net Vin renamed VIN_LAB
Changed lines of the file:
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@@
 		)
 	)
-	(hierarchical_label "Vin"
+	(hierarchical_label "VIN_LAB"
 		(shape output)
 		(at 162.56 52.07 0)
