File: schematics/LIA-board/DAC.kicad_sch (KiCad schematic)
At the start: 21 parts, among them IC1 INA190, IC3 INA190, U10 OPA2196xD, U8 DAC80508, U9 OPA2196xD

Commit message: changes to scematic
Connections:
- net GMOS_Imeas0 renamed IHTR_A
- net GMOS_Imeas1 renamed IHTR_B
- net GMOS_Vadj0 renamed HTR_A
- net GMOS_Vadj1 renamed HTR_B
- net GMOS_Vadj2 renamed DRN_A
- net GMOS_Vadj3 renamed DRN_B
- net GMOS_Vadj4 renamed GATE_DC_A
- net GMOS_Vadj5 renamed GATE_DC_B
- net dac_cs renamed DAC_CS
- net spi_clk renamed SPI_SCK
- net spi_miso renamed SPI_MISO
- net spi_mosi renamed SPI_MOSI
Changed lines of the file:
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@@
 		)
 	)
-	(label "GMOS_Vadj4"
+	(label "GATE_DC_A"
 		(at 160.02 38.1 0)
 		(effects
@@
 		)
 	)
-	(label "GMOS_Vadj5"
+	(label "GATE_DC_B"
 		(at 160.02 40.64 0)
 		(effects
@@
 		)
 	)
-	(label "GMOS_Imeas1"
+	(label "IHTR_B"
 		(at 130.81 101.6 180)
 		(effects
@@
 		)
 	)
-	(label "GMOS_Vadj2"
+	(label "DRN_A"
 		(at 207.01 85.09 0)
 		(effects
@@
 		)
 	)
-	(label "GMOS_Imeas0"
+	(label "IHTR_A"
 		(at 130.81 140.97 180)
 		(effects
@@
 		)
 	)
-	(label "GMOS_Vadj3"
+	(label "DRN_B"
 		(at 207.01 124.46 0)
 		(effects
@@
 		)
 	)
-	(label "GMOS_Vadj1"
+	(label "HTR_B"
 		(at 95.25 85.09 0)
 		(effects
@@
 		)
 	)
-	(label "GMOS_Vadj0"
+	(label "HTR_A"
 		(at 95.25 124.46 0)
 		(effects
@@
 		)
 	)
-	(hierarchical_label "GMOS_Imeas[0..1]"
+	(hierarchical_label "{IHTR_A IHTR_B}"
 		(shape output)
 		(at 256.54 95.25 0)
@@
 		)
 	)
-	(hierarchical_label "spi_miso"
+	(hierarchical_label "SPI_MISO"
 		(shape output)
 		(at 114.3 35.56 180)
@@
 		)
 	)
-	(hierarchical_label "spi_clk"
+	(hierarchical_label "SPI_SCK"
 		(shape input)
 		(at 114.3 30.48 180)
@@
 		)
 	)
-	(hierarchical_label "GMOS_Vadj[0..5]"
+	(hierarchical_label "{HTR_A HTR_B DRN_A DRN_B GATE_DC_A GATE_DC_B}"
 		(shape output)
 		(at 256.54 121.92 0)
@@
 		)
 	)
-	(hierarchical_label "dac_cs"
+	(hierarchical_label "DAC_CS"
 		(shape input)
 		(at 114.3 33.02 180)
@@
 		)
 	)
-	(hierarchical_label "spi_mosi"
+	(hierarchical_label "SPI_MOSI"
 		(shape input)
 		(at 114.3 27.94 180)
