File: schematics/LIA-board/EXCITATION.kicad_sch (KiCad schematic)
At the start: 17 parts, among them U1 OPA2196xD

Commit message: changes to scematic
Connections:
- net Exct0 renamed GATE_B
- net Exct1 renamed GATE_A
- net ext0_vadj renamed GATE_DC_B
- net ext1_vadj renamed GATE_DC_A
- net mcu_sin renamed EXC_DAC
Changed lines of the file:
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@@
 		)
 	)
-	(label "Exct1"
+	(label "GATE_A"
 		(at 182.88 127 0)
 		(effects
@@
 		)
 	)
-	(label "Exct0"
+	(label "GATE_B"
 		(at 182.88 55.88 0)
 		(effects
@@
 		)
 	)
-	(hierarchical_label "Exct[0..1]"
+	(hierarchical_label "{GATE_A GATE_B}"
 		(shape output)
 		(at 199.39 46.99 0)
@@
 		)
 	)
-	(hierarchical_label "ext1_vadj"
+	(hierarchical_label "GATE_DC_A"
 		(shape input)
 		(at 119.38 144.78 180)
@@
 		)
 	)
-	(hierarchical_label "mcu_sin"
+	(hierarchical_label "EXC_DAC"
 		(shape input)
 		(at 119.38 124.46 180)
@@
 		)
 	)
-	(hierarchical_label "mcu_sin"
+	(hierarchical_label "EXC_DAC"
 		(shape input)
 		(at 119.38 53.34 180)
@@
 		)
 	)
-	(hierarchical_label "ext0_vadj"
+	(hierarchical_label "GATE_DC_B"
 		(shape input)
 		(at 119.38 73.66 180)
