File: schematics/LIA-board/GMOS-LIA.kicad_sch (KiCad schematic)
At the start: 0 parts

Commit message: changes to scematic
Other:
- sheet ADC: file adc.kicad_sch -> ADC.kicad_sch
- sheet ADC ports: added ADC_CS, SPI_MISO, SPI_MOSI, SPI_SCK; removed adc_cs, spi_clk, spi_miso, spi_mosi
- sheet Analog: file Analog.kicad_sch -> ANALOG.kicad_sch
- sheet Analog ports: added DRN_A, DRN_B, EXC_DAC, GATE_DC_A, GATE_DC_B, HTR_A, HTR_B, MUX_EN, REF_X, REF_Y, X_OUT, Y_OUT, {MUXA_A0 MUXA_A1 MUXB_A0 MUXB_A1}; removed Vdrain_active, Vdrain_blind, Vheater_active, Vheater_blind, X_chop, X_readout, Y_chop, Y_readout, ch_sel_[0..3], ext0_vadj, ext1_vadj, mcu_sin_ref, mux_en
- sheet Connectors: file connectors.kicad_sch -> CONNECTORS.kicad_sch
- sheet Connectors ports: added VIN_LAB; removed Vin
- sheet DAC: file dac.kicad_sch -> DAC.kicad_sch
- sheet DAC ports: added DAC_CS, SPI_MISO, SPI_MOSI, SPI_SCK, {HTR_A HTR_B DRN_A DRN_B GATE_DC_A GATE_DC_B}, {IHTR_A IHTR_B}; removed GMOS_Imeas[0..1], GMOS_Vadj[0..5], dac_cs, spi_clk, spi_miso, spi_mosi
- sheet DC ports: added I2C_SCL, I2C_SDA, VIN_LAB; removed Vin, i2c_scl, i2c_sda
- sheet MCU: file mcu.kicad_sch -> MCU.kicad_sch
- sheet MCU ports: added EXC_DAC, I2C_SCL, I2C_SDA, SPI_MISO, SPI_MOSI, SPI_SCK, {IHTR_A IHTR_B}; removed V_imeas[0..1], mcu_i2c_scl, mcu_i2c_sda, mcu_sin_ref, spi_miso, spi_mosi, spi_sck
Changed lines of the file:
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@@
 		)
 	)
-	(label "spi_miso"
+	(label "SPI_MISO"
 		(at 210.82 63.5 180)
 		(effects
@@
 		)
 	)
-	(label "spi_clk"
+	(label "SPI_SCK"
 		(at 107.95 64.77 180)
 		(effects
@@
 		)
 	)
-	(label "spi_clk"
+	(label "SPI_SCK"
 		(at 151.13 172.72 0)
 		(effects
@@
 		)
 	)
-	(label "spi_miso"
+	(label "SPI_MISO"
 		(at 151.13 165.1 0)
 		(effects
@@
 		)
 	)
-	(label "GMOS_Vadj1"
+	(label "HTR_B"
 		(at 144.78 86.36 0)
 		(effects
@@
 		)
 	)
-	(label "GMOS_Vadj4"
+	(label "GATE_DC_A"
 		(at 144.78 68.58 0)
 		(effects
@@
 		)
 	)
-	(label "spi_mosi"
+	(label "SPI_MOSI"
 		(at 210.82 67.31 180)
 		(effects
@@
 		)
 	)
-	(label "spi_miso"
+	(label "SPI_MISO"
 		(at 107.95 68.58 180)
 		(effects
@@
 		)
 	)
-	(label "spi_mosi"
+	(label "SPI_MOSI"
 		(at 151.13 168.91 0)
 		(effects
@@
 		)
 	)
-	(label "GMOS_Vadj5"
+	(label "GATE_DC_B"
 		(at 144.78 63.5 0)
 		(effects
@@
 		)
 	)
-	(label "spi_mosi"
+	(label "SPI_MOSI"
 		(at 107.95 72.39 180)
 		(effects
@@
 		)
 	)
-	(label "GMOS_Vadj3"
+	(label "DRN_B"
 		(at 144.78 76.2 0)
 		(effects
@@
 		)
 	)
-	(label "GMOS_Vadj2"
+	(label "DRN_A"
 		(at 144.78 81.28 0)
 		(effects
@@
 		)
 	)
-	(label "spi_clk"
+	(label "SPI_SCK"
 		(at 210.82 59.69 180)
 		(effects
@@
 		)
 	)
-	(label "GMOS_Vadj0"
+	(label "HTR_A"
 		(at 144.78 91.44 0)
 		(effects
@@
 			)
 		)
-		(property "Sheetfile" "Analog.kicad_sch"
+		(property "Sheetfile" "ANALOG.kicad_sch"
 			(at 163.83 147.9046 0)
 			(show_name no)
@@
 			)
 		)
-		(pin "X_readout" output
+		(pin "X_OUT" output
 			(at 196.342 63.5 0)
 			(effects
@@
 			)
 		)
-		(pin "Y_readout" output
+		(pin "Y_OUT" output
 			(at 196.342 68.58 0)
 			(effects
@@
 			)
 		)
-		(pin "mcu_sin_ref" input
+		(pin "EXC_DAC" input
 			(at 163.83 129.54 180)
 			(effects
@@
 			)
 		)
-		(pin "Vdrain_active" input
+		(pin "DRN_B" input
 			(at 163.83 76.2 180)
 			(effects
@@
 			)
 		)
-		(pin "Vdrain_blind" input
+		(pin "DRN_A" input
 			(at 163.83 81.28 180)
 			(effects
@@
 			)
 		)
-		(pin "Vheater_active" input
+		(pin "HTR_B" input
 			(at 163.83 86.36 180)
 			(effects
@@
 			)
 		)
-		(pin "Vheater_blind" input
+		(pin "HTR_A" input
 			(at 163.83 91.44 180)
 			(effects
@@
 			)
 		)
-		(pin "X_chop" input
+		(pin "REF_X" input
 			(at 163.83 139.7 180)
 			(effects
@@
 			)
 		)
-		(pin "Y_chop" input
+		(pin "REF_Y" input
 			(at 163.83 144.78 180)
 			(effects
@@
 			)
 		)
-		(pin "ch_sel_[0..3]" input
+		(pin "{MUXA_A0 MUXA_A1 MUXB_A0 MUXB_A1}" input
 			(at 163.83 119.38 180)
 			(effects
@@
 			)
 		)
-		(pin "mux_en" input
+		(pin "MUX_EN" input
 			(at 163.83 124.46 180)
 			(effects
@@
 			)
 		)
-		(pin "ext0_vadj" input
+		(pin "GATE_DC_B" input
 			(at 163.83 63.5 180)
 			(effects
@@
 			)
 		)
-		(pin "ext1_vadj" input
+		(pin "GATE_DC_A" input
 			(at 163.83 68.58 180)
 			(effects
@@
 			)
 		)
-		(property "Sheetfile" "mcu.kicad_sch"
+		(property "Sheetfile" "MCU.kicad_sch"
 			(at 113.03 178.3846 0)
 			(show_name no)
@@
 			)
 		)
-		(pin "V_imeas[0..1]" input
+		(pin "{IHTR_A IHTR_B}" input
 			(at 113.03 121.92 180)
 			(effects
@@
 			)
 		)
-		(pin "mcu_i2c_scl" tri_state
+		(pin "I2C_SCL" tri_state
 			(at 146.05 154.94 0)
 			(effects
@@
 			)
 		)
-		(pin "mcu_i2c_sda" tri_state
+		(pin "I2C_SDA" tri_state
 			(at 146.05 160.02 0)
 			(effects
@@
 			)
 		)
-		(pin "spi_miso" input
+		(pin "SPI_MISO" input
 			(at 146.05 165.1 0)
 			(effects
@@
 			)
 		)
-		(pin "spi_mosi" output
+		(pin "SPI_MOSI" output
 			(at 146.05 168.91 0)
 			(effects
@@
 			)
 		)
-		(pin "spi_sck" output
+		(pin "SPI_SCK" output
 			(at 146.05 172.72 0)
 			(effects
@@
 			)
 		)
-		(pin "mcu_sin_ref" output
+		(pin "EXC_DAC" output
 			(at 146.05 129.54 0)
 			(effects
@@
 			)
 		)
-		(property "Sheetfile" "dac.kicad_sch"
+		(property "Sheetfile" "DAC.kicad_sch"
 			(at 113.03 107.2646 0)
 			(show_name no)
@@
 			)
 		)
-		(pin "GMOS_Imeas[0..1]" output
+		(pin "{IHTR_A IHTR_B}" output
 			(at 138.43 101.6 0)
 			(effects
@@
 			)
 		)
-		(pin "GMOS_Vadj[0..5]" output
+		(pin "{HTR_A HTR_B DRN_A DRN_B GATE_DC_A GATE_DC_B}" output
 			(at 138.43 95.25 0)
 			(effects
@@
 			)
 		)
-		(pin "dac_cs" input
+		(pin "DAC_CS" input
 			(at 113.03 76.2 180)
 			(effects
@@
 			)
 		)
-		(pin "spi_clk" input
+		(pin "SPI_SCK" input
 			(at 113.03 64.77 180)
 			(effects
@@
 			)
 		)
-		(pin "spi_miso" output
+		(pin "SPI_MISO" output
 			(at 113.03 68.58 180)
 			(effects
@@
 			)
 		)
-		(pin "spi_mosi" input
+		(pin "SPI_MOSI" input
 			(at 113.03 72.39 180)
 			(effects
@@
 			)
 		)
-		(pin "i2c_scl" bidirectional
+		(pin "I2C_SCL" bidirectional
 			(at 246.38 50.8 270)
 			(effects
@@
 			)
 		)
-		(pin "i2c_sda" bidirectional
+		(pin "I2C_SDA" bidirectional
 			(at 250.19 50.8 270)
 			(effects
@@
 			)
 		)
-		(pin "Vin" input
+		(pin "VIN_LAB" input
 			(at 78.74 24.13 180)
 			(effects
@@
 			)
 		)
-		(property "Sheetfile" "connectors.kicad_sch"
+		(property "Sheetfile" "CONNECTORS.kicad_sch"
 			(at 38.1 170.7646 0)
 			(show_name no)
@@
 			)
 		)
-		(pin "Vin" output
+		(pin "VIN_LAB" output
 			(at 63.5 24.13 0)
 			(effects
@@
 			)
 		)
-		(property "Sheetfile" "adc.kicad_sch"
+		(property "Sheetfile" "ADC.kicad_sch"
 			(at 215.9 102.1846 0)
 			(show_name no)
@@
 			)
 		)
-		(pin "adc_cs" input
+		(pin "ADC_CS" input
 			(at 215.9 71.12 180)
 			(effects
@@
 			)
 		)
-		(pin "spi_clk" input
+		(pin "SPI_SCK" input
 			(at 215.9 59.69 180)
 			(effects
@@
 			)
 		)
-		(pin "spi_miso" output
+		(pin "SPI_MISO" output
 			(at 215.9 63.5 180)
 			(effects
@@
 			)
 		)
-		(pin "spi_mosi" input
+		(pin "SPI_MOSI" input
 			(at 215.9 67.31 180)
 			(effects
