File: schematics/LIA-board/LIA_FE.kicad_sch (KiCad schematic)
At the start: 32 parts, among them U2 INA828, U3 OPA2196xD, U4 OPA2196xD, U5 AD630ARZ, U6 AD630ARZ

Commit message: changes to scematic
Connections:
- net Vmid renamed VMID
- net X_chop renamed REF_X
- net X_readout renamed X_OUT
- net Y_chop renamed REF_Y
- net Y_readout renamed Y_OUT
- net active_readout renamed DRN_B
- net blind_readout renamed DRN_A
- net readout renamed BPF_OUT
Changed lines of the file:
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@@
 		)
 	)
-	(label "readout"
+	(label "BPF_OUT"
 		(at 21.59 115.57 0)
 		(effects
@@
 		)
 	)
-	(label "readout"
+	(label "BPF_OUT"
 		(at 151.13 115.57 0)
 		(effects
@@
 		)
 	)
-	(label "Vmid"
+	(label "VMID"
 		(at 31.75 168.91 0)
 		(effects
@@
 		)
 	)
-	(label "Vmid"
+	(label "VMID"
 		(at 161.29 130.81 180)
 		(effects
@@
 		)
 	)
-	(label "readout"
+	(label "BPF_OUT"
 		(at 228.6 52.07 0)
 		(effects
@@
 		)
 	)
-	(label "Vmid"
+	(label "VMID"
 		(at 30.48 130.81 180)
 		(effects
@@
 		)
 	)
-	(hierarchical_label "X_readout"
+	(hierarchical_label "X_OUT"
 		(shape output)
 		(at 139.7 118.11 0)
@@
 		)
 	)
-	(hierarchical_label "blind_readout"
+	(hierarchical_label "DRN_A"
 		(shape input)
 		(at 50.8 57.15 180)
@@
 		)
 	)
-	(hierarchical_label "X_chop"
+	(hierarchical_label "REF_X"
 		(shape input)
 		(at 30.48 125.73 180)
@@
 		)
 	)
-	(hierarchical_label "active_readout"
+	(hierarchical_label "DRN_B"
 		(shape input)
 		(at 50.8 41.91 180)
@@
 		)
 	)
-	(hierarchical_label "Y_chop"
+	(hierarchical_label "REF_Y"
 		(shape input)
 		(at 161.29 125.73 180)
@@
 		)
 	)
-	(hierarchical_label "Y_readout"
+	(hierarchical_label "Y_OUT"
 		(shape output)
 		(at 271.78 118.11 0)
