File: schematics/LIA-board/MCU.kicad_sch (KiCad schematic)
At the start: 9 parts, among them U11 ISO6721BD, U12 STM32U575RGTx, Y1 16MHz

Commit message: changes to scematic
Connections:
- net V_imeas0 renamed IHTR_A
- net V_imeas1 renamed IHTR_B
- net mcu_i2c_scl renamed I2C_SCL
- net mcu_i2c_sda renamed I2C_SDA
- net mcu_sin_ref renamed EXC_DAC
- net spi_miso renamed SPI_MISO
- net spi_mosi renamed SPI_MOSI
- net spi_sck renamed SPI_SCK
Changed lines of the file:
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@@
 	)
 	(bus_entry
-		(at 113.03 72.39)
+		(at 127 72.39)
 		(size 2.54 2.54)
 		(stroke
@@
 	)
 	(bus_entry
-		(at 113.03 69.85)
+		(at 127 69.85)
 		(size 2.54 2.54)
 		(stroke
@@
 	(wire
 		(pts
-			(xy 115.57 72.39) (xy 143.51 72.39)
-		)
-		(stroke
-			(width 0)
-			(type default)
-		)
-	)
-	(wire
-		(pts
-			(xy 115.57 74.93) (xy 143.51 74.93)
+			(xy 129.54 72.39) (xy 143.51 72.39)
+		)
+		(stroke
+			(width 0)
+			(type default)
+		)
+	)
+	(wire
+		(pts
+			(xy 129.54 74.93) (xy 143.51 74.93)
 		)
 		(stroke
@@
 	(bus
 		(pts
-			(xy 113.03 55.88) (xy 113.03 72.39)
+			(xy 127 63.5) (xy 127 72.39)
 		)
 		(stroke
@@
 	(bus
 		(pts
-			(xy 104.14 55.88) (xy 113.03 55.88)
+			(xy 121.92 63.5) (xy 127 63.5)
 		)
 		(stroke
@@
 		)
 	)
-	(label "V_imeas1"
+	(label "IHTR_B"
 		(at 143.51 74.93 180)
 		(effects
@@
 		)
 	)
-	(label "V_imeas0"
+	(label "IHTR_A"
 		(at 143.51 72.39 180)
 		(effects
@@
 		)
 	)
-	(hierarchical_label "mcu_i2c_sda"
+	(hierarchical_label "I2C_SDA"
 		(shape tri_state)
 		(at 190.5 113.03 0)
@@
 		)
 	)
-	(hierarchical_label "spi_mosi"
+	(hierarchical_label "SPI_MOSI"
 		(shape output)
 		(at 190.5 69.85 0)
@@
 		)
 	)
-	(hierarchical_label "mcu_sin_ref"
+	(hierarchical_label "EXC_DAC"
 		(shape output)
 		(at 190.5 62.23 0)
@@
 		)
 	)
-	(hierarchical_label "V_imeas[0..1]"
+	(hierarchical_label "{IHTR_A IHTR_B}"
 		(shape input)
-		(at 104.14 55.88 180)
+		(at 121.92 63.5 180)
 		(effects
 			(font
@@
 		)
 	)
-	(hierarchical_label "spi_miso"
+	(hierarchical_label "SPI_MISO"
 		(shape input)
 		(at 190.5 67.31 0)
@@
 		)
 	)
-	(hierarchical_label "mcu_i2c_scl"
+	(hierarchical_label "I2C_SCL"
 		(shape tri_state)
 		(at 190.5 110.49 0)
@@
 		)
 	)
-	(hierarchical_label "spi_sck"
+	(hierarchical_label "SPI_SCK"
 		(shape output)
 		(at 190.5 54.61 0)
