File: schematics/LIA-board/REGULATORS.kicad_sch (KiCad schematic)
At the start: 38 parts, among them U14 ADP7118ACPZN, U15 LMR51430, U16 ADP7118ACPZN, U17 ADP7118ACPZN, U18 LMR51430, U19 LT3094xMSE, U22 ADP7118ACPZN

Commit message: changes to scematic
Connections:
- net Vin renamed VIN
Changed lines of the file:
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@@
 		)
 	)
-	(hierarchical_label "Vin"
+	(hierarchical_label "VIN"
 		(shape input)
 		(at 36.83 43.18 180)
