File: schematics/LIA-board/USB_PD.kicad_sch (KiCad schematic)
At the start: 15 parts, among them Q1 AO3407A, U13 STUSB4500QTR

Commit message: changes to scematic
Connections:
- net i2c_scl renamed I2C_SCL
- net i2c_sda renamed I2C_SDA
- net usb_pd_alert renamed PD_ALERT
Changed lines of the file:
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@@
 		)
 	)
-	(hierarchical_label "i2c_sda"
+	(hierarchical_label "I2C_SDA"
 		(shape tri_state)
 		(at 217.17 123.19 0)
@@
 		)
 	)
-	(hierarchical_label "i2c_scl"
+	(hierarchical_label "I2C_SCL"
 		(shape tri_state)
 		(at 217.17 119.38 0)
@@
 		)
 	)
-	(hierarchical_label "usb_pd_alert"
+	(hierarchical_label "PD_ALERT"
 		(shape output)
 		(at 217.17 130.81 0)
