File: schematics/LIA-Readout/GMOS_MUX.kicad_sch (KiCad schematic)
At the start: 8 parts, among them J3 DIP40_J19, U20 TMUX1109PW, U21 TMUX1109PW

Commit message: now we are ready to let claude generate AFE schematic
Parts:
- U20, U21: symbol device_libraries:TMUX1109PW -> device_libraries:TMUX1109_TSSOP
Changed lines of the file:
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@@
 	)
 	(symbol
-		(lib_id "device_libraries:TMUX1109PW")
+		(lib_id "device_libraries:TMUX1109_TSSOP")
 		(at 62.23 74.93 0)
 		(mirror y)
@@
 	)
 	(symbol
-		(lib_id "device_libraries:TMUX1109PW")
+		(lib_id "device_libraries:TMUX1109_TSSOP")
 		(at 62.23 153.67 0)
 		(mirror y)
