File: schematics/LIA-AFE-Eval/CONNECTORS.kicad_sch (KiCad schematic)
At the start: 0 parts

Commit message: moving some things in schematic
Parts:
- added C65: 10u, Capacitor_SMD:C_0805_2012Metric, symbol Device:C
- added C66: 100n, Capacitor_SMD:C_0603_1608Metric, symbol Device:C
- added H1, H2, H3, H4: MountingHole_M3, MountingHole:MountingHole_3.2mm_M3, symbol Mechanical:MountingHole
- added J10: X/Y out, Connector_PinHeader_2.54mm:PinHeader_1x05_P2.54mm_Vertical, symbol Connector_Generic:Conn_01x05
- added J7: DC3-2.54-26PAL, Connector_IDC:IDC-Header_2x13_P2.54mm_Horizontal, symbol Connector_Generic:Conn_02x13_Odd_Even
- added J8, J9: SMA, Connector_Coaxial:SMA_Amphenol_132134_Vertical, symbol Connector:Conn_Coaxial
- added TP10: +3V3, TestPoint:TestPoint_Keystone_5000-5004_Miniature, symbol Connector:TestPoint
- added TP11: GND, TestPoint:TestPoint_Keystone_5000-5004_Miniature, symbol Connector:TestPoint
- added TP31: X_OUT, TestPoint:TestPoint_Keystone_5000-5004_Miniature, symbol Connector:TestPoint
- added TP32: Y_OUT, TestPoint:TestPoint_Keystone_5000-5004_Miniature, symbol Connector:TestPoint
- added TP7: EXC_DAC, TestPoint:TestPoint_Keystone_5000-5004_Miniature, symbol Connector:TestPoint
- added TP8: REF_X, TestPoint:TestPoint_Keystone_5000-5004_Miniature, symbol Connector:TestPoint
- added TP9: REF_Y, TestPoint:TestPoint_Keystone_5000-5004_Miniature, symbol Connector:TestPoint
Connections:
- new net +3V3: C65.1, C66.1, J7.25 (Pin_25), J7.26 (Pin_26), TP10.1
- new net DAC_CS: J7.11 (Pin_11)
- new net DSENSE_A: J7.19 (Pin_19)
- new net DSENSE_B: J7.20 (Pin_20)
- new net EXC_DAC: J7.2 (Pin_2), TP7.1
- new net GND: C65.2, C66.2, J10.2 (Pin_2), J10.4 (Pin_4), J7.1 (Pin_1), J7.12 (Pin_12), J7.18 (Pin_18), J7.23 (Pin_23), J7.24 (Pin_24), J7.5 (Pin_5), J7.7 (Pin_7), J8.2 (Ext), J9.2 (Ext), TP11.1
- new net HSENSE_A: J7.21 (Pin_21)
- new net HSENSE_B: J7.22 (Pin_22)
- new net MUXA_A0: J7.13 (Pin_13)
- new net MUXA_A1: J7.14 (Pin_14)
- new net MUXB_A0: J7.15 (Pin_15)
- new net MUXB_A1: J7.16 (Pin_16)
- new net MUX_EN: J7.17 (Pin_17)
- new net REF_X: J7.4 (Pin_4), TP8.1
- new net REF_Y: J7.6 (Pin_6), TP9.1
- new net SPI_MISO: J7.10 (Pin_10)
- new net SPI_MOSI: J7.9 (Pin_9)
- new net SPI_SCLK: J7.8 (Pin_8)
- new net VMID: J10.5 (Pin_5)
- new net X_OUT: TP31.1
- new net X_SMA: J10.1 (Pin_1), J8.1 (In)
- new net Y_OUT: TP32.1
- new net Y_SMA: J10.3 (Pin_3), J9.1 (In)
Other:
- note added: "+3V3 comes from the NUCLEO (DC-4) and supplies DAC80508 VIO and the INA190s."
- note added: "Mounting holes M3, four corners (LU-2)"
- note added: "NUCLEO control header (IF-5): keyed 2 × 13 IDC box header, ribbon wire n = pin n"
- note added: "Test loops: excitation input, references, post-filter outputs, NUCLEO supply (LU-1)"
- note added: "X / Y outputs (IF-3): SMA for the scope and a 1 × 5 header (X, GND, Y, GND, VMID)"
- note removed: "Lab I/O: sensor connection, excitation and reference inputs, X/Y outputs, test points."
- title: Connectors -> Connectors: NUCLEO control header, X/Y outputs, test loops
