File: schematics/LIA-AFE-Eval/DAC.kicad_sch (KiCad schematic)
At the start: 0 parts

Commit message: moving some things in schematic
Parts:
- added C67: 10u, Capacitor_SMD:C_0805_2012Metric, symbol Device:C
- added C68, C69: 100n, Capacitor_SMD:C_0603_1608Metric, symbol Device:C
- added C70: 150n, Capacitor_SMD:C_0603_1608Metric, symbol Device:C
- added U8: DAC80508ZRTET, Package_DFN_QFN:WQFN-16-1EP_3x3mm_P0.5mm_EP1.68x1.68mm, symbol CERN:DAC80508ZRTE
Connections:
- new net +3V3: C69.1, U8.16 (VIO)
- new net +5VA: C67.1, C68.1, U8.7 (VDD)
- new net DAC0: U8.2 (OUT0)
- new net DAC1: U8.3 (OUT1)
- new net DAC2: U8.4 (OUT2)
- new net DAC3: U8.5 (OUT3)
- new net DAC6: U8.10 (OUT6)
- new net DAC7: U8.11 (OUT7)
- new net DAC_CS: U8.12 (~{CS})
- new net DAC_REF: C70.1, U8.1 (REF)
- new net GATE_DC_A: U8.8 (OUT4)
- new net GATE_DC_B: U8.9 (OUT5)
- new net GND: C67.2, C68.2, C69.2, C70.2, U8.17 (EP), U8.6 (GND)
- new net SPI_MISO: U8.15 (SDO/~{ALARM})
- new net SPI_MOSI: U8.14 (SDI)
- new net SPI_SCLK: U8.13 (SCLK)
Other:
- note added: "C70 on REF: 150 nF is an ASSUMPTION, check against the DAC80508 datasheet (REF pin decoupling). OUT0/1 heater A/B, OUT2/3 drain coarse A/B, OUT4/5 gate DC A/B, OUT6/7 drain fine A/B."
- note added: "DAC80508 (U8): AVDD = +5VA, VIO = NUCLEO +3V3, internal 2.5 V reference. Channels as LIA-Readout §4.6.1"
- note removed: "Bias voltages for the sensor (optional on this board)."
- title: DAC -> Bias DAC: DAC80508 (AN-6)
