File: schematics/LIA-AFE-Eval/DEMODULATOR.kicad_sch (KiCad schematic)
At the start: 0 parts

Commit message: moving some things in schematic
Parts:
- added C13: 1.5u, Capacitor_SMD:C_1206_3216Metric, symbol Device:C
- added C94: 150n, Capacitor_SMD:C_1206_3216Metric, symbol Device:C
- added C95, C96: 1u, Capacitor_SMD:C_0603_1608Metric, symbol Device:C
- added C97, C98: 100n, Capacitor_SMD:C_0603_1608Metric, symbol Device:C
- added R14: 200k, Resistor_SMD:R_0603_1608Metric, symbol Device:R
- added R15: 301k, Resistor_SMD:R_0603_1608Metric, symbol Device:R
- added R78, R79: 10k, Resistor_SMD:R_0603_1608Metric, symbol Device:R
- added R80: 100, Resistor_SMD:R_0603_1608Metric, symbol Device:R
- added R81, R82: 10, Resistor_SMD:R_0603_1608Metric, symbol Device:R
- added TP27: DEM_OUT, TestPoint:TestPoint_Keystone_5000-5004_Miniature, symbol Connector:TestPoint
- added TP28: GND, TestPoint:TestPoint_Keystone_5000-5004_Miniature, symbol Connector:TestPoint
- added U24: TMUX6136PWR, Package_SO:TSSOP-16_4.4x5mm_P0.65mm, symbol CERN:TMUX6136PW
- added U26: OPA2196IDGKR, Package_SO:VSSOP-8_3x3mm_P0.65mm, symbol Amplifier_Operational:OPA2196xDGK
Connections:
- new net: R78.2, R79.1, U26.2 (-)
- new net: R14.1, R79.2, TP27.1, U26.1
- new net: U24.3 (D1), U26.3 (+)
- new net +5VA: C97.1, U26.8 (V+)
- new net +9V: R81.1
- new net -5VA: C98.2, U26.4 (V-)
- new net -9V: R82.2
- new net BPF_OUT: R78.1, U24.2 (S1A)
- new net GND: C95.2, C96.1, C97.2, C98.1, TP28.1, U24.4 (S1B), U24.6 (GND), U24.9 (SEL2)
- new net OUT: C13.2, C94.2, R15.2, R80.1, U26.7
- new net OUT_SMA: R80.2
- new net PF_N: C13.1, C94.1, R14.2, R15.1, U26.6 (-)
- new net REF: U24.1 (SEL1)
- new net VDD_SW: C95.1, R81.2, U24.13 (VDD)
- new net VMID_PF: U26.5 (+)
- new net VSS_SW: C96.2, R82.1, U24.5 (VSS)
- no-connect marks 0 -> 8
Other:
- note added: "Post-filter: R_IN 200 kΩ, R_F 301 kΩ ∥ C_F 1.5 µF film (τ = 0.45 s), +IN = VMID_PF; output 100 Ω to SMA/header (AN-12)"
- note added: "Switch demodulator: SEL = 1 → S1A = BPF_OUT (gain +1), SEL = 0 → S1B = GND (gain -1). Second switch unused (E-7)"
- note added: "TMUX6136 supplied from the protected ±9 V input through 10 Ω + 1 µF per pin (DC-3). Truth table: TMUX6136 datasheet SCDS397B Table 6-1."
- note removed: "Synchronous demodulator and post-filter, one channel. This file is used twice (Demod_X, Demod_Y): edit it once, both channels change."
- title: Demodulator (Demod_X, Demod_Y) -> Demodulator (Demod_X, Demod_Y): TMUX6136 + OPA2196, gain ±1, post-filter -1.5, τ = 0.45 s
