File: schematics/LIA-AFE-Eval/EXCITATION.kicad_sch (KiCad schematic)
At the start: 0 parts

Commit message: moving some things in schematic
Parts:
- added C1, C6: 22n, Capacitor_SMD:C_0805_2012Metric, symbol Device:C
- added C2, C4: 100n, Capacitor_SMD:C_0603_1608Metric, symbol Device:C
- added C3, C7: 47n, Capacitor_SMD:C_1206_3216Metric, symbol Device:C
- added C5, C8: 1u, Capacitor_SMD:C_0603_1608Metric, symbol Device:C
- added R1, R3, R5, R7: 1k, Resistor_SMD:R_0603_1608Metric, symbol Device:R
- added R2, R6: 120k, Resistor_SMD:R_0603_1608Metric, symbol Device:R
- added R4, R8: 10k, Resistor_SMD:R_0603_1608Metric, symbol Device:R
- added R58, R59: 100, Resistor_SMD:R_0603_1608Metric, symbol Device:R
- added TP12: GATE_A, TestPoint:TestPoint_Keystone_5000-5004_Miniature, symbol Connector:TestPoint
- added TP13: GATE_B, TestPoint:TestPoint_Keystone_5000-5004_Miniature, symbol Connector:TestPoint
- added TP14: GND, TestPoint:TestPoint_Keystone_5000-5004_Miniature, symbol Connector:TestPoint
- added U1: OPA2196IDGKR, Package_SO:VSSOP-8_3x3mm_P0.65mm, symbol Amplifier_Operational:OPA2196xDGK
Connections:
- new net: C3.1, R1.1, R2.2, R3.1
- new net: C5.1, R4.2, U1.3 (+)
- new net +5VA: C2.1, U1.8 (V+)
- new net -5VA: C4.2, U1.4 (V-)
- new net EXC_DAC: R2.1, R6.1
- new net EXC_NA: C6.1, R7.2, U1.6 (-)
- new net EXC_NB: C1.1, R3.2, U1.2 (-)
- new net EXC_PA: C8.1, R8.2, U1.5 (+)
- new net EXC_XA: C7.1, R5.1, R6.2, R7.1
- new net GATE_A: R59.2, TP12.1
- new net GATE_B: R58.2, TP13.1
- new net GATE_DC_A: R8.1
- new net GATE_DC_B: R4.1
- new net GA_DRV: C6.2, R5.2, R59.1, U1.7
- new net GB_DRV: C1.2, R1.2, R58.1, U1.1
- new net GND: C2.2, C3.2, C4.1, C5.2, C7.2, C8.2, TP14.1
Other:
- note added: "C3/C7 and C1/C6: C0G ±5 % for the first build, rework to ±1 % later (E-5)."
- note added: "Stage A: U1B → GATE_A (pixels 1-3)"
- note added: "Stage B: U1A → GATE_B (pixels 4-6). Gain -1/120 on EXC_DAC, ×1.0083 on GATE_DC_B, f0 = 4.95 kHz"
- note removed: "Gate excitation drive."
- title: Excitation -> Excitation: split-gate MFB summing stages (AN-3)
