File: schematics/LIA-AFE-Eval/FRONT_END.kicad_sch (KiCad schematic)
At the start: 0 parts

Commit message: moving some things in schematic
Parts:
- added C10, C11, C12, C9: 33n, Capacitor_SMD:C_0805_2012Metric, symbol Device:C
- added C88, C89, C90, C91, C92, C93: 100n, Capacitor_SMD:C_0603_1608Metric, symbol Device:C
- added R10: 5.62k, Resistor_SMD:R_0603_1608Metric, symbol Device:R
- added R11, R12, R13, R9: 9.31k, Resistor_SMD:R_0603_1608Metric, symbol Device:R
- added R70, R71, R72, R73, R74, R75: 10k, Resistor_SMD:R_0603_1608Metric, symbol Device:R
- added R76: 150k, Resistor_SMD:R_0603_1608Metric, symbol Device:R
- added R77: 100k, Resistor_SMD:R_0603_1608Metric, symbol Device:R
- added TP22: INA_OUT, TestPoint:TestPoint_Keystone_5000-5004_Miniature, symbol Connector:TestPoint
- added TP23: HPF_OUT, TestPoint:TestPoint_Keystone_5000-5004_Miniature, symbol Connector:TestPoint
- added TP24: BPF_OUT, TestPoint:TestPoint_Keystone_5000-5004_Miniature, symbol Connector:TestPoint
- added TP25: VMID, TestPoint:TestPoint_Keystone_5000-5004_Miniature, symbol Connector:TestPoint
- added TP26: GND, TestPoint:TestPoint_Keystone_5000-5004_Miniature, symbol Connector:TestPoint
- added U2: INA828IDR, Package_SO:SOIC-8_3.9x4.9mm_P1.27mm, symbol CERN:INA828
- added U3: OPA2196IDGKR, Package_SO:VSSOP-8_3x3mm_P0.65mm, symbol Amplifier_Operational:OPA2196xDGK
Connections:
- new net: R11.1, R70.1, R9.2, TP23.1, U3.1
- new net: C9.1, R11.2, R12.1
- new net: C10.1, TP22.1, U2.6 (VO)
- new net: C10.2, C11.1, R9.1
- new net: R10.1, U2.1 (RG)
- new net: R10.2, U2.8 (RG)
- new net: R72.2, R73.1, U3.6 (-)
- new net: C12.1, R12.2, U3.5 (+)
- new net: C11.2, R13.1, U3.3 (+)
- new net: R70.2, R71.1, U3.2 (-)
- new net +5VA: C88.1, C90.1, R74.1, U2.7 (V+), U3.8 (V+)
- new net -5VA: C89.2, C91.2, U2.4 (V-), U3.4 (V-)
- new net BPF_OUT: C9.2, R72.1, TP24.1, U3.7
- new net DRN_A: U2.2 (VIN-)
- new net DRN_B: U2.3 (VIN+)
- new net GND: C12.2, C88.2, C89.1, C90.2, C91.1, C92.2, C93.2, R13.2, R71.2, R73.2, R75.2, R77.2, TP26.1, U2.5 (REF)
- new net VMID: C92.1, R74.2, R75.1, R76.1, TP25.1
- new net VMID_PF: C93.1, R76.2, R77.1
Other:
- note added: "33 nF C0G ±5 % for the first build, rework to ±1 % later (E-5)."
- note added: "ASSUMPTION: divider values (10k/10k, 150k/100k 0.1 %) are not given in the docs. X_OUT/Y_OUT centre on 2.5·VMID_PF = VMID, independent of the VMID loading, because VMID_PF is derived from VMID."
- note added: "Band-pass U3: equal-component Sallen-Key HPF (U3A) + LPF (U3B), R 9.31 kΩ, C 33 nF, K = 2 (Q = 1), ×4 total (AN-7)"
- note added: "In-amp U2: INA828, R_G 5.62 kΩ → G = 9.90 (AN-8). -IN = DRN_A (active), +IN = DRN_B (blind), REF = GND"
- note added: "VMID (2.5 V) and post-filter reference VMID_PF = VMID / 2.5 (LIA-Readout §4.9 FE-B)"
- note removed: "In-amp (differential conversion) and band-pass filter."
- title: Front End -> Front end FE-B: INA828 G = 9.90, Sallen-Key band-pass 518 Hz, VMID
