File: schematics/LIA-AFE-Eval/LIA-AFE-Eval.kicad_sch (KiCad schematic)
At the start: 0 parts

Commit message: moving some things in schematic
Other:
- sheet Connectors ports: added DAC_CS, DSENSE_A, DSENSE_B, EXC_DAC, HSENSE_A, HSENSE_B, MUXA_A0, MUXA_A1, MUXB_A0, MUXB_A1, MUX_EN, REF_X, REF_Y, SPI_MISO, SPI_MOSI, SPI_SCLK, VMID, X_OUT, X_SMA, Y_OUT, Y_SMA; removed none
- sheet DAC ports: added DAC0, DAC1, DAC2, DAC3, DAC6, DAC7, DAC_CS, GATE_DC_A, GATE_DC_B, SPI_MISO, SPI_MOSI, SPI_SCLK; removed none
- sheet Demod_X ports: added BPF_OUT, OUT, OUT_SMA, REF, VMID_PF; removed none
- sheet Demod_Y ports: added BPF_OUT, OUT, OUT_SMA, REF, VMID_PF; removed none
- sheet Excitation ports: added EXC_DAC, GATE_A, GATE_B, GATE_DC_A, GATE_DC_B; removed none
- sheet Front_End ports: added BPF_OUT, DRN_A, DRN_B, VMID, VMID_PF; removed none
- sheet Sensor ports: added DAC0, DAC1, DAC2, DAC3, DAC6, DAC7, DRN_A, DRN_B, DSENSE_A, DSENSE_B, GATE_A, GATE_B, HSENSE_A, HSENSE_B, MUXA_A0, MUXA_A1, MUXB_A0, MUXB_A1, MUX_EN; removed none
- note added: "Root sheet: sheet symbols and inter-sheet wiring only (labels of the same name connect). Rails are global power symbols. Pages follow the sheets left to right, top to bottom."
- note removed: "Root sheet: sheet symbols and inter-sheet wiring only. Pages follow the sheets left to right, top to bottom."
