File: schematics/LIA-AFE-Eval/POWER.kicad_sch (KiCad schematic)
At the start: 0 parts

Commit message: moving some things in schematic
Parts:
- added C40: 10u, Capacitor_SMD:C_0805_2012Metric, symbol Device:C
- added C43: 4.7u, Capacitor_SMD:C_0805_2012Metric, symbol Device:C
- added C52, C54: 10u, Capacitor_SMD:C_1206_3216Metric, symbol Device:C
- added C53, C55, C57, C59, C61, C63, C64: 100n, Capacitor_SMD:C_0603_1608Metric, symbol Device:C
- added C56, C60: 1u, Capacitor_SMD:C_0603_1608Metric, symbol Device:C
- added C58, C62: 2.2u, Capacitor_SMD:C_0603_1608Metric, symbol Device:C
- added D1, D2, D4, D9: B5819W, Diode_SMD:D_SOD-123, symbol Device:D_Schottky
- added J4: WJ500V-5.08-03P, TerminalBlock_Phoenix:TerminalBlock_Phoenix_MKDS-1,5-3-5.08_1x03_P5.08mm_Horizontal, symbol Connector:Screw_Terminal_01x03
- added R37: 49.9k, Resistor_SMD:R_0603_1608Metric, symbol Device:R
- added TP1: +9V, TestPoint:TestPoint_Keystone_5000-5004_Miniature, symbol Connector:TestPoint
- added TP2: -9V, TestPoint:TestPoint_Keystone_5000-5004_Miniature, symbol Connector:TestPoint
- added TP3: +5VA, TestPoint:TestPoint_Keystone_5000-5004_Miniature, symbol Connector:TestPoint
- added TP4: -5VA, TestPoint:TestPoint_Keystone_5000-5004_Miniature, symbol Connector:TestPoint
- added TP5: +5VP, TestPoint:TestPoint_Keystone_5000-5004_Miniature, symbol Connector:TestPoint
- added TP6: GND, TestPoint:TestPoint_Keystone_5000-5004_Miniature, symbol Connector:TestPoint
- added U14, U16: ADP7118ACPZN5.0-R7, Package_CSP:LFCSP-6-1EP_2x2mm_P0.65mm_EP1x1.6mm, symbol Regulator_Linear:ADP7118ACPZN
- added U19: LT3094EMSE#PBF, Package_SO:MSOP-12-1EP_3x4.039mm_P0.65mm_EP1.651x2.845mm, symbol Regulator_Linear:LT3094xMSE
Connections:
- new net: C43.1, R37.1, U19.8 (SET)
- new net +5VA: C58.1, C59.1, D1.1 (K), TP3.1, U16.1 (VOUT), U16.2 (SENSE/ADJ)
- new net +5VP: C62.1, C63.1, TP5.1, U14.1 (VOUT), U14.2 (SENSE/ADJ)
- new net +9V: C52.1, C53.1, C56.1, C57.1, C60.1, C61.1, D4.1 (K), TP1.1, U14.4 (EN), U14.6 (VIN), U16.4 (EN), U16.6 (VIN)
- new net -5VA: C40.2, C64.2, D2.2 (A), TP4.1, U19.10 (OUTS), U19.11 (OUT), U19.12 (OUT)
- new net -9V: C54.2, C55.2, D9.2 (A), TP2.1, U19.1 (IN), U19.13 (IN), U19.2 (IN), U19.3 (EN/UV), U19.5 (PGFB)
- new net GND: C40.1, C43.2, C52.2, C53.2, C54.1, C55.1, C56.2, C57.2, C58.2, C59.2, C60.2, C61.2, C62.2, C63.2, C64.1, D1.2 (A), D2.1 (K), J4.2 (Pin_2), R37.2, TP6.1, U14.3 (GND), U14.7 (GND), U16.3 (GND), U16.7 (GND), U19.6 (ILIM), U19.9 (GND)
- new net VIN_N: D9.1 (K), J4.3 (Pin_3)
- new net VIN_P: D4.2 (A), J4.1 (Pin_1)
- no-connect marks 0 -> 3
Other:
- note added: "+5VA (U16) and +5VP heater rail (U14): ADP7118-5.0 (DC-1, DC-5)"
- note added: "+9V / -9V are the protected inputs (nominal ±9 V, range ±8 to ±12 V). They also supply the TMUX6136 (DC-3)."
- note added: "-5VA: LT3094 (U19), R_SET 49.9 kΩ → -4.99 V; EN/UV and PGFB to IN, ILIM to GND, PG and VIOC open"
- note added: "Input: dual lab supply, reverse-polarity protection (DC-2)"
- note added: "Rail clamps (LIA-Readout DC-4a) and rail test loops (LU-1)"
- note removed: "Bench supply input, protection and the analog rails."
- title: Power -> Power: bench input, protection, analog rails
