File: schematics/LIA-AFE-Eval/SENSOR.kicad_sch (KiCad schematic)
At the start: 0 parts

Commit message: moving some things in schematic
Parts:
- added C71, C72, C73, C76, C77, C80, C81, C82, C83, C84, C85, C86, C87: 100n, Capacitor_SMD:C_0603_1608Metric, symbol Device:C
- added C74, C75: 10u, Capacitor_SMD:C_0805_2012Metric, symbol Device:C
- added C78, C79: 1u, Capacitor_SMD:C_0603_1608Metric, symbol Device:C
- added IC1, IC3: INA190A1IDDFR, Package_TO_SOT_SMD:SOT-23-8, symbol device_libraries:INA190AxDDF
- added J3: DIP-40 socket, Package_DIP:DIP-40_W15.24mm_Socket, symbol device_libraries:DIP40_J19
- added R20, R22, R26, R28: 49.9k, Resistor_SMD:R_0603_1608Metric, symbol Device:R
- added R21, R27, R64, R67: 10k, Resistor_SMD:R_0603_1608Metric, symbol Device:R
- added R23, R29, R38: 100k, Resistor_SMD:R_0603_1608Metric, symbol Device:R
- added R24, R30: 15, Resistor_SMD:R_0603_1608Metric, symbol Device:R
- added R25, R31: 330k, Resistor_SMD:R_0603_1608Metric, symbol Device:R
- added R54, R55: 18k, Resistor_SMD:R_0603_1608Metric, symbol Device:R
- added R56, R57: 1k, Resistor_SMD:R_0805_2012Metric, symbol Device:R
- added R60, R61, R68, R69: 1k, Resistor_SMD:R_0603_1608Metric, symbol Device:R
- added R62, R65: 7.15k, Resistor_SMD:R_0402_1005Metric, symbol Device:R
- added R63, R66: 1.02k, Resistor_SMD:R_0402_1005Metric, symbol Device:R
- added TP15: DRN_A, TestPoint:TestPoint_Keystone_5000-5004_Miniature, symbol Connector:TestPoint
- added TP16: DRN_B, TestPoint:TestPoint_Keystone_5000-5004_Miniature, symbol Connector:TestPoint
- added TP17: VSUP_A, TestPoint:TestPoint_Keystone_5000-5004_Miniature, symbol Connector:TestPoint
- added TP18: VSUP_B, TestPoint:TestPoint_Keystone_5000-5004_Miniature, symbol Connector:TestPoint
- added TP19: HTR_A, TestPoint:TestPoint_Keystone_5000-5004_Miniature, symbol Connector:TestPoint
- added TP20: HTR_B, TestPoint:TestPoint_Keystone_5000-5004_Miniature, symbol Connector:TestPoint
- added TP21: GND, TestPoint:TestPoint_Keystone_5000-5004_Miniature, symbol Connector:TestPoint
- added U10, U23, U9: OPA2196IDGKR, Package_SO:VSSOP-8_3x3mm_P0.65mm, symbol Amplifier_Operational:OPA2196xDGK
- added U20, U21: TMUX1109RSVR, Package_DFN_QFN:UQFN-16_1.8x2.6mm_P0.4mm, symbol device_libraries:TMUX1109_UQFN
Connections:
- new net: J3.14 (NC), J3.26 (NC), J3.27 (NC), J3.34 (NC), J3.35 (NC), J3.7 (NC)
- new net +3V3: C85.1, C87.1, IC1.1 (VS), IC1.2 (ENABLE), IC3.1 (VS), IC3.2 (ENABLE)
- new net +5VA: C71.1, C72.1, C73.1, C76.1, C80.1, J3.15 (VDD), J3.36 (VDD), U10.8 (V+), U20.12 (VDD), U21.12 (VDD), U23.8 (V+)
- new net +5VP: C82.1, U9.8 (V+)
- new net -5VA: C77.2, C81.2, C83.2, U10.4 (V-), U23.4 (V-), U9.4 (V-)
- new net CAL_A: R54.1, U20.5 (S4A)
- new net CAL_B: R55.1, U21.5 (S4A)
- new net DAC0: U9.5 (+)
- new net DAC1: U9.3 (+)
- new net DAC2: U10.3 (+)
- new net DAC3: U10.5 (+)
- new net DAC6: R23.2
- new net DAC7: R29.2
- new net DRN_A: R25.1, TP15.1, U20.6 (DA), U23.3 (+)
- new net DRN_B: R31.1, TP16.1, U21.6 (DA), U23.5 (+)
- new net DSENSE_A: C78.1, R64.2
- new net DSENSE_B: C79.1, R67.2
- new net DS_NA: R21.2, R23.1, U10.2 (-)
- new net DS_NB: R27.2, R29.1, U10.6 (-)
- new net DS_OA: R21.1, R60.1, U10.1
- new net DS_OB: R27.1, R61.1, U10.7
- new net DUMMY_A: R57.1, U20.8 (S4B)
- new net DUMMY_B: R56.1, U21.8 (S4B)
- new net GATE_A: J3.12 (G1), J3.40 (G3), J3.5 (G2)
- new net GATE_B: J3.19 (G6), J3.24 (G5), J3.32 (G4)
- new net GND: C71.2, C72.2, C73.2, C74.2, C75.2, C76.2, C77.1, C78.2, C79.2, C80.2, C81.1, C82.2, C83.1, C84.2, C85.2, C86.2, C87.2, IC1.3 (REF), IC1.4 (GND), IC3.3 (REF), IC3.4 (GND), J3.1 (S3), J3.13 (S1), J3.16 (HN1), J3.2 (HN3), J3.20 (S6), J3.21 (HN6), J3.25 (S5), J3.28 (GND), J3.29 (HN5), J3.33 (S4), J3.37 (HN4), J3.6 (S2), J3.8 (GND), J3.9 (HN2), R22.2, R28.2, R38.2, R54.2, R55.2, R56.2, R57.2, R63.2, R66.2, TP21.1, U20.1 (VSS), U20.13 (GND), U21.1 (VSS), U21.13 (GND)
- new net HSENSE_A: C84.1, R68.2
- new net HSENSE_B: C86.1, R69.2
- new net HTR_A: IC3.8 (IN-), R26.1, R30.2, TP19.1, U20.7 (DB)
- new net HTR_B: IC1.8 (IN-), R20.1, R24.2, TP20.1, U21.7 (DB)
- new net HT_NA: R26.2, R28.1, U9.6 (-)
- new net HT_NB: R20.2, R22.1, U9.2 (-)
- new net HT_OA: IC3.7 (IN+), R30.1, U9.7
- new net HT_OB: IC1.7 (IN+), R24.1, U9.1
- new net IHTR_A: IC3.5 (OUT), R68.1
- new net IHTR_B: IC1.5 (OUT), R69.1
- new net MUXA_A0: U20.15 (A0)
- new net MUXA_A1: U20.14 (A1)
- new net MUXB_A0: U21.15 (A0)
- new net MUXB_A1: U21.14 (A1)
- new net MUX_EN: R38.1, U20.16 (EN), U21.16 (EN)
- new net PIX_D1: J3.17 (D1), U20.2 (S1A)
- new net PIX_D2: J3.10 (D2), U20.3 (S2A)
- new net PIX_D3: J3.3 (D3), U20.4 (S3A)
- new net PIX_D4: J3.38 (D4), U21.2 (S1A)
- new net PIX_D5: J3.30 (D5), U21.3 (S2A)
- new net PIX_D6: J3.22 (D6), U21.4 (S3A)
- new net PIX_H1: J3.11 (HP1), U20.11 (S1B)
- new net PIX_H2: J3.4 (HP2), U20.10 (S2B)
- new net PIX_H3: J3.39 (HP3), U20.9 (S3B)
- new net PIX_H4: J3.31 (HP4), U21.11 (S1B)
- new net PIX_H5: J3.23 (HP5), U21.10 (S2B)
- new net PIX_H6: J3.18 (HP6), U21.9 (S3B)
- new net SN_NA: R62.2, R63.1, U23.2 (-)
- new net SN_NB: R65.2, R66.1, U23.6 (-)
- new net SN_OA: R62.1, R64.1, U23.1
- new net SN_OB: R65.1, R67.1, U23.7
- new net VSUP_A: C74.1, R25.2, R60.2, TP17.1
- new net VSUP_B: C75.1, R31.2, R61.2, TP18.1
Other:
- note added: "Drain sense U23: ×8 (7.15 kΩ / 1.02 kΩ), RC 10 kΩ + 1 µF → DSENSE_A/B to the NUCLEO ADC (IF-4)"
- note added: "Drain supply U10 (V = 1.1·coarse − 0.1·fine), RC 1 kΩ + 10 µF, R_D 330 kΩ (AN-4, AN-4a: ±10 ppm/°C)"
- note added: "GMOS socket J3 (pin map LIA-Readout §1.3) and pixel selection U20 (active 1-3) / U21 (blind 4-6), E-3, E-6"
- note added: "Heater drivers U9 (gain 2, Kelvin feedback after the 15 Ω shunt) and current sense INA190A1 IC3/IC1 (AN-5)"
- note added: "Position 11 (A1 A0): R_CAL R54/R55 on bank A, dummy heater R57/R56 on bank B (AN-13). MUX_EN pull-down R38: all off at reset."
- note added: "R25/R31: matched pair from one reel. Nothing else than U20/U21 DA, the in-amp and the drain-sense input on DRN_A/DRN_B."
- note added: "Test loops (LU-1)"
- note removed: "GMOS socket, pixel selection, drain bias and heater."
- title: Sensor -> Sensor: GMOS socket, pixel selection, drain bias, heaters
